Commit message: modified turtlebot3_waffle urdf to fix sphere radius

File: src/turtlebot3_multi_robot/urdf/turtlebot3_waffle.urdf (robot description, URDF)
Before this commit: robot turtlebot3_waffle, 13 links, 12 joints
Links:
- link caster_back_left_link: geometry collision sphere radius=0.035000
- link caster_back_right_link: geometry collision sphere radius=0.035000
